Commit message: 12 8 2026

File: install/gim_arm_description/share/gim_arm_description/urdf/gim_arm.urdf (robot description, URDF)
Before this commit: robot gim_arm, 6 links, 5 joints
Links:
- link base_link: mass 6.6731 -> 6.66855777151619
- link lower_arm_link: mass 0.586 -> 0.846776609767109
- link shoulder_link: mass 0.06547 -> 0.190732966677201
- link upper_arm_link: mass 2.524 -> 1.15563310050408
Joints:
- joint base_joint: axis 0 0 -1 -> 0.99932 -0.031099 -0.019999; limit lower=0 upper=1.57 effort=5.0 velocity=12.5 -> lower=0 upper=1.57 effort=5 velocity=12.5; origin xyz=0.12249 0 0.13463 rpy=0 -0.17453 0 -> xyz=0.031381 -0.48621 0.64846 rpy=1.4637 1.364 1.4753
- joint elbow_joint: axis 0 0 1 -> 0 0 -1; limit lower=-1.57 upper=0 effort=5.0 velocity=12.5 -> lower=-1.6983 upper=1.1929 effort=5 velocity=12.5; origin xyz=0.21367 -0.052381 -0.02 rpy=0 0 -0.59584 -> xyz=-0.014232 0 -0.21358 rpy=-1.5708 1.1931 0
- joint shoulder_joint: axis 0 0 -1 -> 0 -1 0; limit lower=-0.2 upper=1.57 effort=5.0 velocity=12.5 -> lower=-1.1811 upper=1.2002 effort=5 velocity=12.5; origin xyz=0 0.098298 -0.082481 rpy=0 1.3963 1.5708 -> xyz=-0.049966 0.001555 0.00099995 rpy=-1.3842 -0.058173 1.7475

File: src/gim_arm_description/urdf/gim_arm.urdf (robot description, URDF)
Before this commit: robot gim_arm, 6 links, 5 joints
Joints:
- joint elbow_joint: axis 0 0 1 -> 0 0 -1; limit lower=0 upper=1.57 effort=5 velocity=12.5 -> lower=-1.6983 upper=1.1929 effort=5 velocity=12.5
- joint shoulder_joint: axis 0 1 0 -> 0 -1 0; limit lower=-0.2 upper=1.57 effort=5 velocity=12.5 -> lower=-1.1811 upper=1.2002 effort=5 velocity=12.5

Commit message: abc

File: install/gim_arm_description/share/gim_arm_description/urdf/gim_arm.urdf (robot description, URDF)
Before this commit: robot gim_arm, 6 links, 5 joints
Joints:
- joint elbow_joint: limit lower=-1.6983 upper=1.1929 effort=5 velocity=12.5 -> lower=-0.6618 upper=1.6104 effort=5 velocity=12.5
- joint shoulder_joint: limit lower=-1.1811 upper=1.2002 effort=5 velocity=12.5 -> lower=-0.9328 upper=1.4388 effort=5 velocity=12.5

File: install/gim_arm_description/share/gim_arm_description/urdf/gim_arm_origin.urdf (robot description, URDF)
Before this commit: robot gim_arm, 6 links, 5 joints
Joints:
- joint elbow_joint: limit lower=-1.6983 upper=1.1929 effort=5 velocity=12.5 -> lower=-0.6618 upper=1.6104 effort=5 velocity=12.5
- joint shoulder_joint: limit lower=-1.1811 upper=1.2002 effort=5 velocity=12.5 -> lower=-0.9328 upper=1.4388 effort=5 velocity=12.5

File: kinematics_test/gim_arm.urdf (robot description, URDF)
Before this commit: robot gim_arm, 6 links, 5 joints
Joints:
- joint elbow_joint: limit lower=-1.6983 upper=1.1929 effort=5 velocity=12.5 -> lower=-0.6618 upper=1.6104 effort=5 velocity=12.5
- joint shoulder_joint: limit lower=-1.1811 upper=1.2002 effort=5 velocity=12.5 -> lower=-0.9328 upper=1.4388 effort=5 velocity=12.5

File: src/gim_arm_mujoco/gim_arm_mujoco.urdf (robot description, URDF)
Before this commit: robot gim_arm, 6 links, 5 joints
Links:
- link base_link: geometry collision mesh filename=/home/minh/gim60108_ws/src/gim_arm_mujoco/meshes/base_link.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; visual mesh filename=/home/minh/gim60108_ws/src/gim_arm_mujoco/meshes/base_link.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
- link lower_arm_link: geometry collision mesh filename=/home/minh/gim60108_ws/src/gim_arm_mujoco/meshes/lower_arm_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; visual mesh filename=/home/minh/gim60108_ws/src/gim_arm_mujoco/meshes/lower_arm_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
- link shoulder_link: geometry collision mesh filename=/home/minh/gim60108_ws/src/gim_arm_mujoco/meshes/shoulder_l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; visual mesh filename=/home/minh/gim60108_ws/src/gim_arm_mujoco/meshes/shoulder_l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
- link upper_arm_link: geometry collision mesh filename=/home/minh/gim60108_ws/src/gim_arm_mujoco/meshes/upper_arm_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; visual mesh filename=/home/minh/gim60108_ws/src/gim_arm_mujoco/meshes/upper_arm_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
Joints:
- joint base_footprint_to_base_link: origin xyz=0 0 0 rpy=0 0 0 -> xyz=0 0 0 rpy=0.083 0 0
- joint elbow_joint: limit lower=0 upper=1.57 effort=5 velocity=12.5 -> lower=-0.6618 upper=1.6104 effort=5 velocity=12.5; origin xyz=-0.014232 0 -0.21358 rpy=-1.5708 1.1931 0 -> xyz=-0.014232 0 -0.21358 rpy=1.570809721 1.469492654 -3.141575913
- joint shoulder_joint: limit lower=-0.2 upper=1.57 effort=5 velocity=12.5 -> lower=-0.9328 upper=1.4388 effort=5 velocity=12.5; origin xyz=-0.049966 0.001555 0.00099995 rpy=-1.3842 -0.058173 1.7475 -> xyz=-0.049966 0.001555 0.00099995 rpy=-1.375708549 0.010247217 1.396947503

Commit message: Revert "abc"
This reverts commit 331fb13cb0f6401638bd860e3db4a7e281926588.

File: install/gim_arm_description/share/gim_arm_description/urdf/gim_arm.urdf (robot description, URDF)
Before this commit: robot gim_arm, 6 links, 5 joints
Joints:
- joint elbow_joint: limit lower=-0.6618 upper=1.6104 effort=5 velocity=12.5 -> lower=-1.6983 upper=1.1929 effort=5 velocity=12.5
- joint shoulder_joint: limit lower=-0.9328 upper=1.4388 effort=5 velocity=12.5 -> lower=-1.1811 upper=1.2002 effort=5 velocity=12.5

File: install/gim_arm_description/share/gim_arm_description/urdf/gim_arm_origin.urdf (robot description, URDF)
Before this commit: robot gim_arm, 6 links, 5 joints
Joints:
- joint elbow_joint: limit lower=-0.6618 upper=1.6104 effort=5 velocity=12.5 -> lower=-1.6983 upper=1.1929 effort=5 velocity=12.5
- joint shoulder_joint: limit lower=-0.9328 upper=1.4388 effort=5 velocity=12.5 -> lower=-1.1811 upper=1.2002 effort=5 velocity=12.5

File: kinematics_test/gim_arm.urdf (robot description, URDF)
Before this commit: robot gim_arm, 6 links, 5 joints
Joints:
- joint elbow_joint: limit lower=-0.6618 upper=1.6104 effort=5 velocity=12.5 -> lower=-1.6983 upper=1.1929 effort=5 velocity=12.5
- joint shoulder_joint: limit lower=-0.9328 upper=1.4388 effort=5 velocity=12.5 -> lower=-1.1811 upper=1.2002 effort=5 velocity=12.5

File: src/gim_arm_mujoco/gim_arm_mujoco.urdf (robot description, URDF)
Before this commit: robot gim_arm, 6 links, 5 joints
Links:
- link base_link: geometry collision mesh filename=meshes/base_link.STL; visual mesh filename=meshes/base_link.STL
- link lower_arm_link: geometry collision mesh filename=meshes/lower_arm_link.STL; visual mesh filename=meshes/lower_arm_link.STL
- link shoulder_link: geometry collision mesh filename=meshes/shoulder_link.STL; visual mesh filename=meshes/shoulder_link.STL
- link upper_arm_link: geometry collision mesh filename=meshes/upper_arm_link.STL; visual mesh filename=meshes/upper_arm_link.STL
Joints:
- joint base_footprint_to_base_link: origin xyz=0 0 0 rpy=0.083 0 0 -> xyz=0 0 0 rpy=0 0 0
- joint elbow_joint: limit lower=-0.6618 upper=1.6104 effort=5 velocity=12.5 -> lower=0 upper=1.57 effort=5 velocity=12.5; origin xyz=-0.014232 0 -0.21358 rpy=1.570809721 1.469492654 -3.141575913 -> xyz=-0.014232 0 -0.21358 rpy=-1.5708 1.1931 0
- joint shoulder_joint: limit lower=-0.9328 upper=1.4388 effort=5 velocity=12.5 -> lower=-0.2 upper=1.57 effort=5 velocity=12.5; origin xyz=-0.049966 0.001555 0.00099995 rpy=-1.375708549 0.010247217 1.396947503 -> xyz=-0.049966 0.001555 0.00099995 rpy=-1.3842 -0.058173 1.7475
