Commit message: Ghi chú ngắn gọn về những gì bạn vừa sửa

File: install/gim_arm_moveit_config/share/gim_arm_moveit_config/config/gim_arm.ros2_control.xacro (robot description, xacro)
@@ -1,33 +1 @@
-<?xml version="1.0"?>
-<robot xmlns:xacro="http://www.ros.org/wiki/xacro">
-    <xacro:macro name="gim_arm_ros2_control" params="name initial_positions_file">
-        <xacro:property name="initial_positions" value="${load_yaml(initial_positions_file)['initial_positions']}"/>
-        <ros2_control name="${name}" type="system">
-            <hardware>
-                <!-- By default, set up controllers for simulation. This won't work on real hardware -->
-                <plugin>mock_components/GenericSystem</plugin>
-            </hardware>
-            <joint name="base_joint">
-                <command_interface name="position"/>
-                <state_interface name="position">
-                  <param name="initial_value">${initial_positions['base_joint']}</param>
-                </state_interface>
-                <state_interface name="velocity"/>
-            </joint>
-            <joint name="shoulder_joint">
-                <command_interface name="position"/>
-                <state_interface name="position">
-                  <param name="initial_value">${initial_positions['shoulder_joint']}</param>
-                </state_interface>
-                <state_interface name="velocity"/>
-            </joint>
-            <joint name="elbow_joint">
-                <command_interface name="position"/>
-                <state_interface name="position">
-                  <param name="initial_value">${initial_positions['elbow_joint']}</param>
-                </state_interface>
-                <state_interface name="velocity"/>
-            </joint>
-        </ros2_control>
-    </xacro:macro>
-</robot>
+/home/minh/git_gim_ws/GIM_Arm_3_DOF/src/gim_arm_moveit_config/config/gim_arm.ros2_control.xacro

File: install/gim_arm_moveit_config/share/gim_arm_moveit_config/config/gim_arm_urdf.xacro (robot description, xacro)
@@ -1,7 +1 @@
-<?xml version="1.0"?>
-<robot xmlns:xacro="http://www.ros.org/wiki/xacro" name="gim_arm">
-    <!-- Import gim_arm urdf file: đã có sẵn <ros2_control name="GimArmSystem">
-         thật (plugin gim_arm_hardware/GimArmSystemHardware) bên trong rồi,
-         không cần và không được thêm block ros2_control giả nào nữa. -->
-    <xacro:include filename="$(find gim_arm_description)/urdf/gim_arm.urdf" />
-</robot>
+/home/minh/git_gim_ws/GIM_Arm_3_DOF/src/gim_arm_moveit_config/config/gim_arm_urdf.xacro
