Commit message: Ghi chú ngắn gọn về những gì bạn vừa sửa

File: kinematics_test/gim_arm_mujoco.urdf (robot description, URDF)
Before this commit: robot gim_arm, 6 links, 5 joints
Joints:
- joint base_footprint_to_base_link: origin xyz=0 0 0 rpy=0 0 0 -> xyz=0 0 0 rpy=0.083 0 0
- joint elbow_joint: origin xyz=-0.014232 0 -0.21358 rpy=-1.5708 1.1931 0 -> xyz=-0.014232 0 -0.21358 rpy=1.570809721 1.469492654 -3.141575913
- joint shoulder_joint: origin xyz=-0.049966 0.001555 0.00099995 rpy=-1.3842 -0.058173 1.7475 -> xyz=-0.049966 0.001555 0.00099995 rpy=-1.375708549 0.010247217 1.396947503
