Commit message: Ghi chú ngắn gọn về những gì bạn vừa sửa

File: kinematics_test/gim_arm.urdf (robot description, URDF)
Before this commit: robot gim_arm, 6 links, 5 joints
Joints:
- joint base_joint: limit lower=0 upper=1.57 effort=5 velocity=12.5 -> lower=0 upper=1.57 effort=5 velocity=15.708
- joint elbow_joint: limit lower=-1.6983 upper=1.1929 effort=5 velocity=12.5 -> lower=-1.6983 upper=1.1929 effort=5 velocity=15.708
- joint shoulder_joint: limit lower=-1.1811 upper=1.2002 effort=5 velocity=12.5 -> lower=-1.1811 upper=1.2002 effort=40 velocity=1.963

File: kinematics_test/gim_arm_mujoco.urdf (robot description, URDF)
Before this commit: robot gim_arm, 6 links, 5 joints
Joints:
- joint base_joint: limit lower=0 upper=1.57 effort=5 velocity=12.5 -> lower=0 upper=1.57 effort=5 velocity=15.708
- joint elbow_joint: limit lower=-1.6983 upper=1.1929 effort=5 velocity=12.5 -> lower=-1.6983 upper=1.1929 effort=5 velocity=15.708
- joint shoulder_joint: limit lower=-1.1811 upper=1.2002 effort=5 velocity=12.5 -> lower=-1.1811 upper=1.2002 effort=40 velocity=1.963

File: src/gim_arm_description/urdf/gim_arm_origin.urdf (robot description, URDF)
Before this commit: robot gim_arm, 6 links, 5 joints
Joints:
- joint base_joint: limit lower=0 upper=1.57 effort=5 velocity=12.5 -> lower=0 upper=1.57 effort=5 velocity=15.708
- joint elbow_joint: limit lower=-1.6983 upper=1.1929 effort=5 velocity=12.5 -> lower=-1.6983 upper=1.1929 effort=5 velocity=15.708
- joint shoulder_joint: limit lower=-1.1811 upper=1.2002 effort=5 velocity=12.5 -> lower=-1.1811 upper=1.2002 effort=40 velocity=1.963

Commit message: 6251

File: kinematics_test/gim_arm.urdf (robot description, URDF)
Before this commit: robot gim_arm, 6 links, 5 joints
Joints:
- joint base_joint: limit lower=0 upper=1.57 effort=5 velocity=15.708 -> lower=-0.7121 upper=1.0226 effort=5 velocity=15.708
- joint elbow_joint: limit lower=-1.6983 upper=1.1929 effort=5 velocity=15.708 -> lower=-0.2336 upper=1.7762 effort=5 velocity=15.708
- joint shoulder_joint: limit lower=-1.1811 upper=1.2002 effort=40 velocity=1.963 -> lower=-0.2366 upper=1.3435 effort=40 velocity=1.963

File: kinematics_test/gim_arm_mujoco.urdf (robot description, URDF)
Before this commit: robot gim_arm, 6 links, 5 joints
Joints:
- joint base_joint: limit lower=0 upper=1.57 effort=5 velocity=15.708 -> lower=-0.7121 upper=1.0226 effort=5 velocity=15.708
- joint elbow_joint: limit lower=-1.6983 upper=1.1929 effort=5 velocity=15.708 -> lower=-0.2336 upper=1.7762 effort=5 velocity=15.708
- joint shoulder_joint: limit lower=-1.1811 upper=1.2002 effort=40 velocity=1.963 -> lower=-0.2366 upper=1.3435 effort=40 velocity=1.963

File: src/gim_arm_description/urdf/gim_arm_origin.urdf (robot description, URDF)
Before this commit: robot gim_arm, 6 links, 5 joints
Joints:
- joint base_joint: limit lower=0 upper=1.57 effort=5 velocity=15.708 -> lower=-0.7121 upper=1.0226 effort=5 velocity=15.708
- joint elbow_joint: limit lower=-1.6983 upper=1.1929 effort=5 velocity=15.708 -> lower=-0.2336 upper=1.7762 effort=5 velocity=15.708
- joint shoulder_joint: limit lower=-1.1811 upper=1.2002 effort=40 velocity=1.963 -> lower=-0.2366 upper=1.3435 effort=40 velocity=1.963

File: src/gim_arm_mujoco/gim_arm_mujoco.urdf (robot description, URDF)
Before this commit: robot gim_arm, 6 links, 5 joints
Joints:
- joint base_joint: limit lower=0 upper=1.57 effort=5 velocity=12.5 -> lower=-0.7121 upper=1.0226 effort=5 velocity=12.5
- joint elbow_joint: limit lower=0 upper=1.57 effort=5 velocity=12.5 -> lower=-0.2336 upper=1.7762 effort=5 velocity=12.5
- joint shoulder_joint: limit lower=-0.2 upper=1.57 effort=5 velocity=12.5 -> lower=-0.2366 upper=1.3435 effort=5 velocity=12.5
