Commit message: Ghi chú về những gì bạn vừa cập nhật

File: src/gim_arm_description/urdf/gim_arm.urdf (robot description, URDF)
Before this commit: robot gim_arm, 6 links, 5 joints
Links:
- link base_link: mass 6.6731 -> 6.66855777151619
- link lower_arm_link: mass 0.586 -> 0.846776609767109
- link shoulder_link: mass 0.06547 -> 0.190732966677201
- link upper_arm_link: mass 2.524 -> 1.15563310050408
Joints:
- joint base_joint: axis 0 0 -1 -> 0.99932 -0.031099 -0.019999; limit lower=0 upper=1.57 effort=5.0 velocity=12.5 -> lower=0 upper=1.57 effort=5 velocity=12.5; origin xyz=0.12249 0 0.13463 rpy=0 -0.17453 0 -> xyz=0.031381 -0.48621 0.64846 rpy=1.4637 1.364 1.4753
- joint elbow_joint: limit lower=-1.57 upper=0 effort=5.0 velocity=12.5 -> lower=0 upper=1.57 effort=5 velocity=12.5; origin xyz=0.21367 -0.052381 -0.02 rpy=0 0 -0.59584 -> xyz=-0.014232 0 -0.21358 rpy=-1.5708 1.1931 0
- joint shoulder_joint: axis 0 0 -1 -> 0 1 0; limit lower=-0.2 upper=1.57 effort=5.0 velocity=12.5 -> lower=-0.2 upper=1.57 effort=5 velocity=12.5; origin xyz=0 0.098298 -0.082481 rpy=0 1.3963 1.5708 -> xyz=-0.049966 0.001555 0.00099995 rpy=-1.3842 -0.058173 1.7475

Commit message: Add modular effort controllers and stabilize Gazebo control

File: src/gim_arm_description/urdf/gim_arm.urdf (robot description, URDF)
Before this commit: robot gim_arm, 6 links, 5 joints
Links:
- link lower_arm_link: mass 0.84674 -> 0.73459
- link upper_arm_link: mass 1.1556 -> 1.2678
